File: assemble/assemble.kicad_sch (KiCad schematic)
At the start: 94 parts, among them J1 Conn_01x04, SW1 SW_Push, SW10 SW_Push, SW11 SW_Push, SW12 SW_Push, SW13 SW_Push, SW14 SW_Push, SW15 SW_Push, SW16 SW_Push, SW17 SW_Push, SW18 SW_Push, SW19 RotaryEncoder_Switch, SW2 SW_Push, SW20 SW_SPDT, SW21 SW_Push, SW22 SW_Push, SW23 SW_Push, SW24 SW_Push, SW25 SW_Push, SW26 SW_Push, SW27 SW_Push, SW28 RotaryEncoder_Switch, SW29 SW_Push, SW3 SW_Push, SW30 SW_Push, SW31 SW_Push, SW32 SW_Push, SW33 SW_Push, SW34 SW_Push, SW35 SW_Push, SW36 SW_Push, SW37 SW_Push, SW38 SW_Push, SW39 SW_Push, SW4 SW_Push, SW40 SW_Push, SW41 SW_Push, SW42 SW_Push, SW43 SW_Push, SW44 SW_Push, SW45 SW_Push, SW46 SW_Push, SW5 SW_Push, SW6 SW_Push, SW7 SW_Push, SW8 SW_Push, SW9 SW_Push

Commit message: feat: add pcb data
Parts:
- SW44: renamed from SW33; footprint kicad-lib:CherryMX-HotSwap-1u_17 -> kbd_Parts:ResetSW
- U1: footprint kicad-lib:AE-XCL102D333CR-G -> kbd_Parts:Micon_BMP_7sKB
- renumbered D23 to D22, D24 to D23, D25 to D24, D26 to D25, D27 to D26, D28 to D27, D29 to D28, D30 to D29, D32 to D30, D33 to D31, D34 to D32, D35 to D33, D36 to D34, D37 to D35, D38 to D36, D39 to D37, D40 to D38, D41 to D39, D42 to D40, D43 to D41, D44 to D42, D22 to D45, D31 to D46, SW21 to SW19, SW22 to SW20, SW23 to SW21, SW24 to SW22, SW25 to SW23, SW26 to SW24, SW27 to SW25, SW29 to SW26, SW30 to SW27, SW31 to SW28, SW32 to SW29, SW34 to SW30, SW35 to SW31, SW36 to SW32, SW37 to SW33, SW38 to SW34, SW39 to SW35, SW40 to SW36, SW41 to SW37, SW42 to SW38, SW43 to SW39, SW44 to SW40, SW45 to SW41, SW46 to SW42, SW19 to SW45, SW28 to SW46, SW20 to SW47
Connections:
- net GND: now also J1.1 (Pin_1); no longer J1.4 (Pin_4)
- net SDA: now also J1.4 (Pin_4); no longer J1.2 (Pin_2)
- net VCC: now also J1.2 (Pin_2); no longer J1.1 (Pin_1)
