File: switch_plate/switch_plate.kicad_sch (KiCad schematic)
At the start: 96 parts, among them J1 Conn_01x04, SW1 SW_Push, SW10 SW_Push, SW11 SW_Push, SW12 SW_Push, SW13 SW_Push, SW14 SW_Push, SW15 SW_Push, SW16 SW_Push, SW17 SW_Push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

Commit message: feat: add switch plate
Parts:
- R1, R2: value R_470k -> R_US; footprint Resistor_THT:R_Axial_DIN0204_L3.6mm_D1.6mm_P5.08mm_Horizontal -> (none)
Other:
- moved on the sheet: J1
