File: switch_plate/switch_plate.kicad_pcb (KiCad board)
At the start: 2 copper layers, 283.6 x 113.2 mm, 50 parts, among them SW1 SW_Push, SW10 SW_Push, SW11 SW_Push, SW12 SW_Push, SW13 SW_Push, SW14 SW_Push, SW15 SW_Push, SW16 SW_Push, SW17 SW_Push, SW18 SW_Push, SW19 SW_Push, SW2 SW_Push, SW20 SW_Push, SW21 SW_Push, SW22 SW_Push, SW23 SW_Push, SW24 SW_Push, SW25 SW_Push, SW26 SW_Push, SW27 SW_Push, SW28 SW_Push, SW29 SW_Push, SW3 SW_Push, SW30 SW_Push, SW31 SW_Push, SW32 SW_Push, SW33 SW_Push, SW34 SW_Push, SW35 SW_Push, SW36 SW_Push, SW37 SW_Push, SW38 SW_Push, SW39 SW_Push, SW4 SW_Push, SW40 SW_Push, SW41 SW_Push, SW42 SW_Push, SW5 SW_Push, SW6 SW_Push, SW7 SW_Push, SW8 SW_Push, SW9 SW_Push

Commit message: feat: change screw
Parts:
- removed REF** (x8): set_screw_hole, kicad-lib:set_screw_hole
- added Ref**: Val**, kbd_Hole:m3_Screw_Hole_EdgeCuts, F.Cu at (126.9, 94.8)
- added Ref**: Val**, kbd_Hole:m3_Screw_Hole_EdgeCuts, F.Cu at (134.5, 134.3)
- added Ref**: Val**, kbd_Hole:m3_Screw_Hole_EdgeCuts, F.Cu at (170.1, 94.8)
- added Ref**: Val**, kbd_Hole:m3_Screw_Hole_EdgeCuts, F.Cu at (162.5, 134.3)
Other:
- outline, holes or cut-outs redrawn

Commit message: fix: footprint
Parts:
- Ref** (x4): footprint kbd_Hole:m3_Screw_Hole_EdgeCuts -> MountingHole:MountingHole_3.2mm_M3
