File: v2/assemble/assemble.kicad_pcb (KiCad board)
At the start: 2 copper layers, 283.6 x 105.3 mm, 96 parts, among them J1 Conn_01x04, SW1 SW_Push, SW10 SW_Push, SW11 SW_Push, SW12 SW_Push, SW13 SW_Push, SW14 SW_Push, SW15 SW_Push, SW16 SW_Push, SW17 SW_Push, SW18 SW_Push, SW19 SW_Push, SW2 SW_Push, SW20 SW_Push, SW21 SW_Push, SW22 SW_Push, SW23 SW_Push, SW24 SW_Push, SW25 SW_Push, SW26 SW_Push, SW27 SW_Push, SW28 SW_Push, SW29 SW_Push, SW3 SW_Push, SW30 SW_Push, SW31 SW_Push, SW32 SW_Push, SW33 SW_Push, SW34 SW_Push, SW35 SW_Push, SW36 SW_Push, SW37 SW_Push, SW38 SW_Push, SW39 SW_Push, SW4 SW_Push, SW40 SW_Push, SW41 SW_Push, SW42 SW_Push, SW44 SW_Push, SW45 RotaryEncoder_Switch, SW46 RotaryEncoder_Switch, SW47 SW_SPDT, SW5 SW_Push, SW6 SW_Push, SW7 SW_Push, SW8 SW_Push, SW9 SW_Push

Commit message: feat: implement v2 pcb
Parts:
- removed D45, D46: D, kbd_Parts:Diode_SMD
- removed SW44: SW_Push, kbd_Parts:ResetSW
- added U4: XIAO-nRF52840-SMD, xiao:XIAO-nRF52840-SMD, B.Cu at (148.5, 44.2)
- R1, R2: footprint Resistor_THT:R_Axial_DIN0204_L3.6mm_D1.6mm_P7.62mm_Horizontal -> Resistor_THT:R_Axial_DIN0204_L3.6mm_D1.6mm_P5.08mm_Horizontal
- U1: value ~ -> XIAO-nRF52840-SMD; footprint kbd_Parts:Micon_BMP_7sKB -> xiao:XIAO-nRF52840-SMD; moved to F.Cu
- moved U1 15.7 mm to (135.8, 44.3), turned to 0 degrees
- moved R2 11.6 mm to (137.5, 89.1), turned to -90 degrees
- moved R1 6.69 mm to (131.8, 89.1), turned to -90 degrees
- moved AE-XCL102D333CR-G1 3.82 mm to (162.5, 62.2)
- moved J1 3.00 mm to (151.3, 91.8)
- turned D30 to 10 degrees
Connections:
- D1 pad 1: ROW1 -> ROW1L
- D10 pad 1: ROW2 -> ROW2L
- D11 pad 1: ROW3 -> ROW3L
- D12 pad 1: ROW4 -> ROW4L
- D13 pad 1: ROW1 -> Net-(D13-K)
- D13 pad 2: Net-(D13-A) -> ROW1L
- D14 pad 1: ROW2 -> Net-(D14-K)
- D14 pad 2: Net-(D14-A) -> ROW2L
- D15 pad 1: ROW3 -> Net-(D15-K)
- D15 pad 2: Net-(D15-A) -> ROW3L
- D16 pad 1: ROW1 -> Net-(D16-K)
- D16 pad 2: Net-(D16-A) -> ROW1L
- D17 pad 1: ROW2 -> Net-(D17-K)
- D17 pad 2: Net-(D17-A) -> ROW2L
- D18 pad 1: ROW3 -> Net-(D18-K)
- D18 pad 2: Net-(D18-A) -> ROW3L
- D19 pad 1: ROW1 -> Net-(D19-K)
- D19 pad 2: Net-(D19-A) -> ROW1L
- D2 pad 1: ROW2 -> ROW2L
- D20 pad 1: ROW2 -> Net-(D20-K)
- D20 pad 2: Net-(D20-A) -> ROW2L
- D21 pad 1: ROW3 -> Net-(D21-K)
- D21 pad 2: Net-(D21-A) -> ROW3L
- D22 pad 2: ROW1 -> ROW1R
- D23 pad 2: ROW2 -> ROW2R
- D24 pad 2: ROW3 -> ROW3R
- D25 pad 2: ROW4 -> ROW4R
- D26 pad 2: ROW1 -> ROW1R
- D27 pad 2: ROW2 -> ROW2R
- D28 pad 2: ROW3 -> ROW3R
- D29 pad 2: ROW4 -> ROW4R
- D3 pad 1: ROW3 -> ROW3L
- D30 pad 2: ROW1 -> ROW1R
- D31 pad 2: ROW2 -> ROW2R
- D32 pad 2: ROW3 -> ROW3R
- D33 pad 2: ROW4 -> ROW4R
- D34 pad 1: Net-(D34-K) -> ROW1R
- D34 pad 2: ROW1 -> Net-(D34-A)
- D35 pad 1: Net-(D35-K) -> ROW2R
- D35 pad 2: ROW2 -> Net-(D35-A)
- D36 pad 1: Net-(D36-K) -> ROW3R
- D36 pad 2: ROW3 -> Net-(D36-A)
- D37 pad 1: Net-(D37-K) -> ROW1R
- D37 pad 2: ROW1 -> Net-(D37-A)
- D38 pad 1: Net-(D38-K) -> ROW2R
- D38 pad 2: ROW2 -> Net-(D38-A)
- D39 pad 1: Net-(D39-K) -> ROW3R
- D39 pad 2: ROW3 -> Net-(D39-A)
- D4 pad 1: ROW4 -> ROW4L
- D40 pad 1: Net-(D40-K) -> ROW1R
- D40 pad 2: ROW1 -> Net-(D40-A)
- D41 pad 1: Net-(D41-K) -> ROW2R
- D41 pad 2: ROW2 -> Net-(D41-A)
- D42 pad 1: Net-(D42-K) -> ROW3R
- D42 pad 2: ROW3 -> Net-(D42-A)
- D5 pad 1: ROW1 -> ROW1L
- D6 pad 1: ROW2 -> ROW2L
- D7 pad 1: ROW3 -> ROW3L
- D8 pad 1: ROW4 -> ROW4L
- D9 pad 1: ROW1 -> ROW1L
- J1 pad 1: GND -> GNDL
- SW1 pad 1: COL1 -> COL1L
- SW10 pad 1: COL3 -> COL3L
- SW11 pad 1: COL3 -> COL3L
- SW12 pad 1: COL3 -> COL3L
- SW13 pad 1: COL4 -> COL1L
- SW13 pad 2: Net-(D13-A) -> Net-(D13-K)
- SW14 pad 1: COL4 -> COL1L
- SW14 pad 2: Net-(D14-A) -> Net-(D14-K)
- SW15 pad 1: COL4 -> COL1L
- SW15 pad 2: Net-(D15-A) -> Net-(D15-K)
- SW16 pad 1: COL5 -> COL2L
- SW16 pad 2: Net-(D16-A) -> Net-(D16-K)
- SW17 pad 1: COL5 -> COL2L
- SW17 pad 2: Net-(D17-A) -> Net-(D17-K)
- SW18 pad 1: COL5 -> COL2L
- SW18 pad 2: Net-(D18-A) -> Net-(D18-K)
- SW19 pad 1: COL6 -> COL3L
- SW19 pad 2: Net-(D19-A) -> Net-(D19-K)
- SW2 pad 1: COL1 -> COL1L
- SW20 pad 1: COL6 -> COL3L
- SW20 pad 2: Net-(D20-A) -> Net-(D20-K)
- SW21 pad 1: COL6 -> COL3L
- SW21 pad 2: Net-(D21-A) -> Net-(D21-K)
- SW22 pad 1: COL1 -> COL1R
- SW23 pad 1: COL1 -> COL1R
- SW24 pad 1: COL1 -> COL1R
- SW25 pad 1: COL1 -> COL1R
- SW26 pad 1: COL2 -> COL2R
- SW27 pad 1: COL2 -> COL2R
- SW28 pad 1: COL2 -> COL2R
- SW29 pad 1: COL2 -> COL2R
- SW3 pad 1: COL1 -> COL1L
- SW30 pad 1: COL3 -> COL3R
- SW31 pad 1: COL3 -> COL3R
- SW32 pad 1: COL3 -> COL3R
- SW33 pad 1: COL3 -> COL3R
- SW34 pad 1: COL4 -> COL1R
- SW34 pad 2: Net-(D34-K) -> Net-(D34-A)
- SW35 pad 1: COL4 -> COL1R
- SW35 pad 2: Net-(D35-K) -> Net-(D35-A)
- SW36 pad 1: COL4 -> COL1R
- SW36 pad 2: Net-(D36-K) -> Net-(D36-A)
- SW37 pad 1: COL5 -> COL2R
- SW37 pad 2: Net-(D37-K) -> Net-(D37-A)
- SW38 pad 1: COL5 -> COL2R
- SW38 pad 2: Net-(D38-K) -> Net-(D38-A)
- SW39 pad 1: COL5 -> COL2R
- SW39 pad 2: Net-(D39-K) -> Net-(D39-A)
- SW4 pad 1: COL1 -> COL1L
- SW40 pad 1: COL6 -> COL3R
- SW40 pad 2: Net-(D40-K) -> Net-(D40-A)
- SW41 pad 1: COL6 -> COL3R
- SW41 pad 2: Net-(D41-K) -> Net-(D41-A)
- SW42 pad 1: COL6 -> COL3R
- SW42 pad 2: Net-(D42-K) -> Net-(D42-A)
- SW45 pad C: GND -> GNDL
- SW45 pad S1: COL4 -> unconnected-(SW45-PadS1)
- SW45 pad S2: Net-(D45-A) -> unconnected-(SW45-PadS2)
- SW46 pad C: GND -> GNDR
- SW46 pad S1: COL5 -> unconnected-(SW46-PadS1)
- SW46 pad S2: Net-(D46-A) -> unconnected-(SW46-PadS2)
- SW5 pad 1: COL2 -> COL2L
- SW6 pad 1: COL2 -> COL2L
- SW7 pad 1: COL2 -> COL2L
- SW8 pad 1: COL2 -> COL2L
- SW9 pad 1: COL3 -> COL3L
- U1 pad 1: unconnected-(U1-D3/PIN1-Pad1) -> RE1A
- U1 pad 10: ROW3 -> ROW2L
- U1 pad 11: ROW4 -> ROW1L
- U1 pad 12: RE1A -> VCC
- U1 pad 13: RE1B -> GNDL
- U1 pad 14: ROW2 -> unconnected-(U1-5V-Pad14)
- U1 pad 15: ROW1 -> BAT+
- U1 pad 16: COL3 -> BAT-
- U1 pad 17: COL2 -> unconnected-(U1-NFC1-Pad17)
- U1 pad 18: COL1 -> unconnected-(U1-NFC2-Pad18)
- U1 pad 19: RE2B -> unconnected-(U1-PA31_SWDIO-Pad19)
- U1 pad 2: unconnected-(U1-D2/PIN2-Pad2) -> RE1B
- U1 pad 20: RE2A -> unconnected-(U1-PA30_SWCLK-Pad20)
- U1 pad 21: VCC -> unconnected-(U1-RESET-Pad21)
- U1 pad 22: RESET -> unconnected-(U1-GND-Pad22)
- U1 pad 3: BAT- -> COL1L
- U1 pad 4: GND -> COL2L
- U1 pad 7: COL4 -> COL3L
- U1 pad 8: COL5 -> ROW4L
- U1 pad 9: COL6 -> ROW3L
Routing:
- net COL6: track 510.6 -> 0.00 mm, vias 11 -> 0
- net COL4: track 458.9 -> 0.00 mm, vias 18 -> 0
- net COL5: track 458.8 -> 0.00 mm, vias 25 -> 0
- net COL3: track 422.3 -> 0.00 mm, vias 23 -> 0
- net ROW1: track 419.8 -> 0.00 mm, vias 32 -> 0
- net ROW2: track 380.9 -> 0.00 mm, vias 24 -> 0
- net ROW3: track 364.1 -> 0.00 mm, vias 19 -> 0
- net GND: track 341.4 -> 0.00 mm, vias 1 -> 0
- net COL2: track 333.6 -> 0.00 mm, vias 22 -> 0
- net ROW4: track 329.0 -> 0.00 mm, vias 17 -> 0
- net COL1: track 301.7 -> 0.00 mm, vias 17 -> 0
- net COL3R: track 0.00 -> 268.7 mm, vias 0 -> 18
- net COL3L: track 0.00 -> 255.7 mm, vias 0 -> 6
- net GNDR: track 0.00 -> 238.8 mm, vias 0 -> 6
- net COL1L: track 0.00 -> 236.8 mm, vias 0 -> 5
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Other:
- board text added: "Orbit One v2.0 Designed by derui"
- board text removed: "Orbit One v1.0 Designed by derui"

Commit message: fix: plot setting
Routing:
- net BAT-: track 89.9 -> 91.0 mm
Changed lines of the file:
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@@
 			(drillshape 0)
 			(scaleselection 1)
-			(outputdirectory "../jclpcb/assemble/")
+			(outputdirectory "../jclpcb/")
 		)
 	)
@@
 		(attr smd)
 		(fp_line
-			(start 2.699998 -0.75)
+			(start 2.699997 -0.75)
 			(end -2.7 -0.75)
 			(stroke
@@
 		(fp_line
 			(start 2.7 0.75)
-			(end 2.699998 -0.75)
+			(end 2.699997 -0.75)
 			(stroke
 				(width 0.15)
@@
 		(fp_line
 			(start -2.7 -0.75)
-			(end -2.699998 0.75)
+			(end -2.699997 0.75)
 			(stroke
 				(width 0.15)
@@
 		)
 		(fp_line
-			(start -2.699998 0.75)
+			(start -2.699997 0.75)
 			(end 2.7 0.75)
 			(stroke
@@
 			(layer "F.SilkS")
 		)
-		(fp_circle
-			(center -9.155 -10.121)
-			(end -9.155 -10.375)
-			(stroke
-				(width 0.5)
-				(type solid)
-			)
-			(fill yes)
-			(layer "F.SilkS")
-		)
-		(fp_circle
-			(center -7.881 -9.404)
-			(end -7.881 -9.658)
-			(stroke
-				(width 0.5)
-				(type solid)
-			)
-			(fill yes)
-			(layer "F.SilkS")
-		)
 		(fp_rect
 			(start -8.945 -10.55)
@@
 			(layer "F.Fab")
 		)
-		(fp_circle
-			(center -7.861 -9.4)
-			(end -7.861 -9.654)
-			(stroke
-				(width 0.5)
-				(type solid)
-			)
-			(fill yes)
-			(layer "F.Fab")
-		)
 		(pad "1" smd roundrect
 			(at -8.11 -7.62)
@@
 		(attr smd)
 		(fp_line
-			(start 2.699998 0.75)
+			(start 2.699997 0.75)
 			(end 2.7 -0.75)
 			(stroke
@@
 		(fp_line
 			(start 2.7 -0.75)
-			(end -2.699998 -0.75)
+			(end -2.699997 -0.75)
 			(stroke
 				(width 0.15)
@@
 		(fp_line
 			(start -2.7 0.75)
-			(end 2.699998 0.75)
+			(end 2.699997 0.75)
 			(stroke
 				(width 0.15)
@@
 		)
 		(fp_line
-			(start -2.699998 -0.75)
+			(start -2.699997 -0.75)
 			(end -2.7 0.75)
 			(stroke
@@
 		(attr smd)
 		(fp_line
-			(start 2.699998 -0.75)
+			(start 2.699997 -0.75)
 			(end -2.7 -0.75)
 			(stroke
@@
 		(fp_line
 			(start 2.7 0.75)
-			(end 2.699998 -0.75)
+			(end 2.699997 -0.75)
 			(stroke
 				(width 0.15)
@@
 		(fp_line
 			(start -2.7 -0.75)
-			(end -2.699998 0.75)
+			(end -2.699997 0.75)
 			(stroke
 				(width 0.15)
@@
 		)
 		(fp_line
-			(start -2.699998 0.75)
+			(start -2.699997 0.75)
 			(end 2.7 0.75)
 			(stroke
@@
 		(attr smd)
 		(fp_line
-			(start 2.699998 -0.75)
+			(start 2.699997 -0.75)
 			(end -2.7 -0.75)
 			(stroke
@@
 		(fp_line
 			(start 2.7 0.75)
-			(end 2.699998 -0.75)
+			(end 2.699997 -0.75)
 			(stroke
 				(width 0.15)
@@
 		(fp_line
 			(start -2.7 -0.75)
-			(end -2.699998 0.75)
+			(end -2.699997 0.75)
 			(stroke
 				(width 0.15)
@@
 		)
 		(fp_line
-			(start -2.699998 0.75)
+			(start -2.699997 0.75)
 			(end 2.7 0.75)
 			(stroke
@@
 		(attr smd)
 		(fp_line
-			(start 2.699998 0.75)
+			(start 2.699997 0.75)
 			(end 2.7 -0.75)
 			(stroke
@@
 		(fp_line
 			(start 2.7 -0.75)
-			(end -2.699998 -0.75)
+			(end -2.699997 -0.75)
 			(stroke
 				(width 0.15)
@@
 		(fp_line
 			(start -2.7 0.75)
-			(end 2.699998 0.75)
+			(end 2.699997 0.75)
 			(stroke
 				(width 0.15)
@@
 		)
 		(fp_line
-			(start -2.699998 -0.75)
+			(start -2.699997 -0.75)
 			(end -2.7 0.75)
 			(stroke
@@
 		(attr smd)
 		(fp_line
-			(start 2.699998 0.75)
+			(start 2.699997 0.75)
 			(end 2.7 -0.75)
 			(stroke
@@
 		(fp_line
 			(start 2.7 -0.75)
-			(end -2.699998 -0.75)
+			(end -2.699997 -0.75)
 			(stroke
 				(width 0.15)
@@
 		(fp_line
 			(start -2.7 0.75)
-			(end 2.699998 0.75)
+			(end 2.699997 0.75)
 			(stroke
 				(width 0.15)
@@
 		)
 		(fp_line
-			(start -2.699998 -0.75)
+			(start -2.699997 -0.75)
 			(end -2.7 0.75)
 			(stroke
@@
 			(layer "B.SilkS")
 		)
-		(fp_circle
-			(center -7.881 9.404)
-			(end -7.881 9.658)
-			(stroke
-				(width 0.5)
-				(type solid)
-			)
-			(fill yes)
-			(layer "B.SilkS")
-		)
-		(fp_circle
-			(center -9.155 10.121)
-			(end -9.155 10.375)
-			(stroke
-				(width 0.5)
-				(type solid)
-			)
-			(fill yes)
-			(layer "B.SilkS")
-		)
 		(fp_rect
 			(start -8.945 10.55)
@@
 			(layer "B.Fab")
 		)
-		(fp_circle
-			(center -7.861 9.4)
-			(end -7.861 9.654)
-			(stroke
-				(width 0.5)
-				(type solid)
-			)
-			(fill yes)
-			(layer "B.Fab")
-		)
 		(pad "1" smd roundrect
 			(at -8.11 7.62 180)
@@
 	)
 	(segment
+		(start 150.4 58.2)
+		(end 150.4 57.4)
+		(width 0.5)
+		(layer "F.Cu")
+		(net 5)
+	)
+	(segment
 		(start 151 42.2)
 		(end 152.8315 42.2)
@@
 	)
 	(segment
-		(start 150.4 58.2)
+		(start 150.4 57.4)
 		(end 150.4 42.8)
 		(width 0.5)
@@
 	(segment
 		(start 150.4 58.2)
-		(end 133.8 58.2)
+		(end 149.6 58.2)
+		(width 0.5)
+		(layer "F.Cu")
+		(net 5)
+	)
+	(segment
+		(start 149.6 58.2)
+		(end 150.4 57.4)
 		(width 0.5)
 		(layer "F.Cu")
@@
 		(width 0.5)
 		(layer "F.Cu")
+		(net 5)
+	)
+	(segment
+		(start 149.6 58.2)
+		(end 133.8 58.2)
+		(width 0.5)
+		(layer "F.Cu")
